File: ksoloti-gills.kicad_pcb (KiCad board)
At the start: 2 copper layers, 150 x 92 mm, 224 parts, among them J1 9-20VDC, J10 MIDI_OUT, J11 MIDI_IO, J12 LINE_IN_OUT, J13 HP_OUT, J14 HP_POT, J15 MIDI1_CFG, J16 EXPANSION, J17 GATE_OUT, J18 MIDI_OUT_GND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

Commit message: Add "CC BY 4.0 Ksoloti" to silkscreens - see README
Other:
- board text added: "CC BY 4.0 Ksoloti"
Changed lines of the file:
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@@
+		)
+	)
+	(gr_text "CC BY 4.0 Ksoloti"
+		(at 69.8952 118.017 90)
+		(layer "F.SilkS")
+		(effects
+			(font
+				(size 1 1)
+				(thickness 0.2)
+				(bold yes)
+			)
 		)
 	)
@@
 			)
 			(justify mirror)
+		)
+	)
+	(gr_text "CC BY 4.0 Ksoloti"
+		(at 69.8952 118.017 270)
+		(layer "B.SilkS")
+		(effects
+			(font
+				(size 1 1)
+				(thickness 0.2)
+				(bold yes)
+			)
+			(justify mirror)
