File: ksoloti-gills-cv-expander/ksoloti-gills-cv-expander.kicad_pcb (KiCad board)
At the start: 2 copper layers, 64 x 20.5 mm, 54 parts, among them J1 EXPANSION, J2 12V_PWR, U1 XL6007, U2 L78L12_SOT89, U3 L79L12_SOT89, U4 CJ431, U5 TL072

Commit message: Add "CC BY 4.0 Ksoloti" to silkscreens - see README
Other:
- board text added: "CC BY 4.0 Ksoloti"
Changed lines of the file:
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@@
 		(tags "SOD-323")
 		(property "Reference" "D2"
-			(at 0.0014 4.46 0)
+			(at 1.272 4.587 0)
 			(layer "F.SilkS")
 			(effects
@@
 		(tags "SOD-323")
 		(property "Reference" "D1"
-			(at -0.0032 -5.222 0)
+			(at -1.2738 -5.349 0)
 			(layer "F.SilkS")
 			(effects
@@
 		(tags "SOD-323")
 		(property "Reference" "D3"
-			(at -0.0014 -5.984 0)
+			(at -1.272 -6.111 0)
 			(layer "F.SilkS")
 			(effects
@@
 		)
 	)
+	(gr_text "CC BY 4.0 Ksoloti"
+		(at 70.1662 61.937 0)
+		(layer "F.SilkS")
+		(effects
+			(font
+				(size 1 1)
+				(thickness 0.2)
+				(bold yes)
+			)
+		)
+	)
+	(gr_text "CC BY 4.0 Ksoloti"
+		(at 70.1662 61.937 -0)
+		(layer "B.SilkS")
+		(effects
+			(font
+				(size 1 1)
+				(thickness 0.2)
+				(bold yes)
+			)
+			(justify mirror)
+		)
+	)
