File: ksoloti-gills_panel/ksoloti-gills_panel.kicad_pcb (KiCad board)
At the start: 2 copper layers, 519 x 352.8 mm, 124 parts

Commit message: Add "CC BY 4.0 Ksoloti" to silkscreens - see README
Other:
- board text added: "CC BY 4.0 Ksoloti"
